File: testAdapter1_2.kicad_pcb (KiCad board)
At the start: 2 copper layers, 64 x 50.1 mm, 48 parts, among them J1 CONN-SCSI68, J2 CONN-SMK20, P1 SDATA+, P10 CTR-, P11 CLK+, P12 CLK-, P13 SDATA4+, P14 SDATA4-, P2 SDATA-, P3 SDATA+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

Commit message: Aktueller Stand
Parts:
- added ?: LOGO, LOGO, F.Cu at (132.8, 88.5)
- P1: value SDATA+ -> SDATA1+
- P2: value SDATA- -> SDATA1-
- P3: value SDATA+ -> SDATA3+
- P9: value CLK+ -> CTR+
Routing:
- net (no net): track 4.50 -> 0.00 mm, vias 1 -> 0
- net GND: track 128.3 -> 125.0 mm, vias 9 -> 10
Other:
- net class Default: via_dia 0.889 -> 0.9144
- net class GND: via_dia 0.889 -> 0.9144
- net class HV: via_dia 0.889 -> 0.9144
- net class Power: via_dia 0.889 -> 0.9144
- board text added: "+"
- board text added: "-"
- board text added: "CLK"
- board text added: "CTR"
- board text added: "FPix to DTB adapter"
- board text added: "GND"
- board text added: "Oct 2013, F. Meier"
- board text added: "SDA"
- board text added: "SDATA1"
- board text added: "SDATA3"
- board text added: "SDATA4"
- board text added: "TOUT"
- board text added: "University of Nebraska, Lincoln"
