File: FPix2DTB_90deg/FPix2DTB_90deg.sch (KiCad schematic (older format))
At the start: 48 parts, among them J1 CONN-SCSI68, J2 CONN-SMK20, P1 SDATA+, P10 CTR-, P11 CLK+, P12 CLK-, P13 SDATA4+, P14 SDATA4-, P2 SDATA-, P3 SDATA+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

Commit message: Weiter
Parts:
- removed P10: CTR-, testpad, symbol TST
- removed P11, P9: CLK+, testpad, symbol TST
- removed P12: CLK-, testpad, symbol TST
- removed P13: SDATA4+, testpad, symbol TST
- removed P14: SDATA4-, testpad, symbol TST
- removed P2: SDATA-, testpad, symbol TST
- removed P3: SDATA+, testpad, symbol TST
- removed P4: SDATA3-, testpad, symbol TST
- removed P5: TOUT+, testpad, symbol TST
- removed P6: TOUT-, testpad, symbol TST
- removed P7: SDA+, testpad, symbol TST
- removed P8: SDA-, testpad, symbol TST
- added P?: RClk-, symbol TST
- added P?: OutA-, symbol TST
- added P?: RClk+, symbol TST
- added P?: RDa+, symbol TST
- added P?: RDa-, symbol TST
- added P?: SDA+, symbol TST
- added P?: SDA-, symbol TST
- added P?: CTR+, symbol TST
- added P?: CTR-, symbol TST
- added P?: CLK+, symbol TST
- added P?: CLK-, symbol TST
- added P?: 160Clk+, symbol TST
- added P?: 160Clk-, symbol TST
- P1: value SDATA+ -> OutA+; footprint testpad -> (none)
- R22, R25, R26: value 10k -> 10k 0.1%
- R23, R24: value 10k -> 10k 5%
Connections:
- net SDATA1_p: no longer P1.1
- net TBM_Out_A+: now also P1.1
Other:
- moved on the sheet: P1

Commit message: Weiter
Parts:
- added P1: VA, symbol TST
- added P18: RTD+, symbol TST
- added P19: RTD-, symbol TST
- added P2: 3V3, symbol TST
- added P20: GND, symbol TST
- added P3: VD, symbol TST
- gave numbers to parts that had none: 13
- renumbered P1 to P4
Connections:
- net 3V3: now also P2.1
- net TBM_160MHz_Out+: now also P16.1
- net TBM_160MHz_Out-: now also P17.1
- net TBM_Clk_In+: now also P14.1
- net TBM_Clk_In-: now also P15.1
- net TBM_Out_A-: now also P5.1
- net TBM_RClk_Out+: now also P6.1
- net TBM_RClk_Out-: now also P7.1
- net TBM_RDa_Out+: now also P8.1
- net TBM_RDa_Out-: now also P9.1
- net TBM_SD_In+: now also P10.1
- net TBM_SD_In-: now also P11.1
- net TBM_Trig_In+: now also P12.1
- net TBM_Trig_In-: now also P13.1
- net VA: now also P1.1
- net VD: now also P3.1
Changed lines of the file:
@@
 $EndComp
 $Comp
-L GND #PWR01
+L GND #PWR9
 U 1 1 526C1DE7
 P 13700 -6750
-F 0 "#PWR01" H 13700 -6750 30  0001 C CNN
+F 0 "#PWR9" H 13700 -6750 30  0001 C CNN
 F 1 "GND" H 13700 -6820 30  0001 C CNN
 F 2 "" H 13700 -6750 60  0000 C CNN
@@
 $EndComp
 $Comp
-L GND #PWR02
+L GND #PWR5
 U 1 1 526C1DF6
 P 3100 5100
-F 0 "#PWR02" H 3100 5100 30  0001 C CNN
+F 0 "#PWR5" H 3100 5100 30  0001 C CNN
 F 1 "GND" H 3100 5030 30  0001 C CNN
 F 2 "" H 3100 5100 60  0000 C CNN
@@
 VD
 $Comp
-L GND #PWR03
+L GND #PWR8
 U 1 1 526C1ECD
 P 10300 6750
-F 0 "#PWR03" H 10300 6750 30  0001 C CNN
+F 0 "#PWR8" H 10300 6750 30  0001 C CNN
 F 1 "GND" H 10300 6680 30  0001 C CNN
 F 2 "" H 10300 6750 60  0000 C CNN
@@
 $EndComp
 $Comp
-L GND #PWR04
+L GND #PWR2
 U 1 1 526C717E
 P 1200 7100
-F 0 "#PWR04" H 1200 7100 30  0001 C CNN
+F 0 "#PWR2" H 1200 7100 30  0001 C CNN
 F 1 "GND" H 1200 7030 30  0001 C CNN
 F 2 "" H 1200 7100 60  0000 C CNN
@@
 NoConn ~ 2800 4500
 $Comp
-L GND #PWR05
+L GND #PWR3
 U 1 1 526C8467
 P 1500 5100
-F 0 "#PWR05" H 1500 5100 30  0001 C CNN
+F 0 "#PWR3" H 1500 5100 30  0001 C CNN
 F 1 "GND" H 1500 5030 30  0001 C CNN
 F 2 "" H 1500 5100 60  0000 C CNN
@@
 Connection ~ 5300 7550
 $Comp
-L GND #PWR06
+L GND #PWR7
 U 1 1 526C8E08
 P 6500 7700
-F 0 "#PWR06" H 6500 7700 30  0001 C CNN
+F 0 "#PWR7" H 6500 7700 30  0001 C CNN
 F 1 "GND" H 6500 7630 30  0001 C CNN
 F 2 "" H 6500 7700 60  0000 C CNN
@@
 	6500 7450 6500 7700
 $Comp
-L GND #PWR07
+L GND #PWR6
 U 1 1 526EC52D
 P 3550 5800
-F 0 "#PWR07" H 3550 5800 30  0001 C CNN
+F 0 "#PWR6" H 3550 5800 30  0001 C CNN
 F 1 "GND" H 3550 5730 30  0001 C CNN
 F 2 "" H 3550 5800 60  0000 C CNN
@@
 $EndComp
 $Comp
-L GND #PWR08
+L GND #PWR1
 U 1 1 526EC987
 P 1050 6050
-F 0 "#PWR08" H 1050 6050 30  0001 C CNN
+F 0 "#PWR1" H 1050 6050 30  0001 C CNN
 F 1 "GND" H 1050 5980 30  0001 C CNN
 F 2 "" H 1050 6050 60  0000 C CNN
@@
 $EndComp
 $Comp
-L GND #PWR09
+L GND #PWR4
 U 1 1 526EC996
 P 1650 6050
-F 0 "#PWR09" H 1650 6050 30  0001 C CNN
+F 0 "#PWR4" H 1650 6050 30  0001 C CNN
 F 1 "GND" H 1650 5980 30  0001 C CNN
 F 2 "" H 1650 6050 60  0000 C CNN
@@
 	1650 5850 1650 6050
 $Comp
-L TST P1
+L TST P4
 U 1 1 526ECC25
 P 6000 800
-F 0 "P1" H 6000 1100 40  0000 C CNN
+F 0 "P4" H 6000 1100 40  0000 C CNN
 F 1 "OutA+" H 6000 1050 30  0000 C CNN
 F 2 "" H 6000 800 60  0000 C CNN
@@
 	5100 800  4850 800
 $Comp
-L TST P?
+L TST P7
 U 1 1 527C410F
 P 6200 2100
-F 0 "P?" H 6200 2400 40  0000 C CNN
+F 0 "P7" H 6200 2400 40  0000 C CNN
 F 1 "RClk-" H 6200 2350 30  0000 C CNN
 F 2 "" H 6200 2100 60  0000 C CNN
@@
 	5600 4500 6400 4500
 $Comp
-L TST P?
+L TST P5
 U 1 1 527C44F9
 P 6200 1300
-F 0 "P?" H 6200 1600 40  0000 C CNN
+F 0 "P5" H 6200 1600 40  0000 C CNN
 F 1 "OutA-" H 6200 1550 30  0000 C CNN
 F 2 "" H 6200 1300 60  0000 C CNN
@@
 $EndComp
 $Comp
-L TST P?
+L TST P6
 U 1 1 527C4508
 P 6000 1600
-F 0 "P?" H 6000 1900 40  0000 C CNN
+F 0 "P6" H 6000 1900 40  0000 C CNN
 F 1 "RClk+" H 6000 1850 30  0000 C CNN
 F 2 "" H 6000 1600 60  0000 C CNN
@@
 $EndComp
 $Comp
-L TST P?
+L TST P8
 U 1 1 527C4517
 P 6000 2400
-F 0 "P?" H 6000 2700 40  0000 C CNN
+F 0 "P8" H 6000 2700 40  0000 C CNN
 F 1 "RDa+" H 6000 2650 30  0000 C CNN
 F 2 "" H 6000 2400 60  0000 C CNN
@@
 $EndComp
 $Comp
-L TST P?
+L TST P9
 U 1 1 527C4530
 P 6200 2900
-F 0 "P?" H 6200 3200 40  0000 C CNN
+F 0 "P9" H 6200 3200 40  0000 C CNN
 F 1 "RDa-" H 6200 3150 30  0000 C CNN
 F 2 "" H 6200 2900 60  0000 C CNN
@@
 $EndComp
 $Comp
-L TST P?
+L TST P10
 U 1 1 527C453F
 P 6000 3200
-F 0 "P?" H 6000 3500 40  0000 C CNN
+F 0 "P10" H 6000 3500 40  0000 C CNN
 F 1 "SDA+" H 6000 3450 30  0000 C CNN
 F 2 "" H 6000 3200 60  0000 C CNN
@@
 $EndComp
 $Comp
-L TST P?
+L TST P11
 U 1 1 527C454E
 P 6200 3700
-F 0 "P?" H 6200 4000 40  0000 C CNN
+F 0 "P11" H 6200 4000 40  0000 C CNN
 F 1 "SDA-" H 6200 3950 30  0000 C CNN
 F 2 "" H 6200 3700 60  0000 C CNN
@@
 $EndComp
 $Comp
-L TST P?
+L TST P12
 U 1 1 527C455D
 P 6000 4000
-F 0 "P?" H 6000 4300 40  0000 C CNN
+F 0 "P12" H 6000 4300 40  0000 C CNN
 F 1 "CTR+" H 6000 4250 30  0000 C CNN
 F 2 "" H 6000 4000 60  0000 C CNN
@@
 $EndComp
 $Comp
-L TST P?
+L TST P13
 U 1 1 527C456C
 P 6200 4500
-F 0 "P?" H 6200 4800 40  0000 C CNN
+F 0 "P13" H 6200 4800 40  0000 C CNN
 F 1 "CTR-" H 6200 4750 30  0000 C CNN
 F 2 "" H 6200 4500 60  0000 C CNN
@@
 $EndComp
 $Comp
-L TST P?
+L TST P14
 U 1 1 527C457B
 P 6000 4800
-F 0 "P?" H 6000 5100 40  0000 C CNN
+F 0 "P14" H 6000 5100 40  0000 C CNN
 F 1 "CLK+" H 6000 5050 30  0000 C CNN
 F 2 "" H 6000 4800 60  0000 C CNN
@@
 $EndComp
 $Comp
-L TST P?
+L TST P15
 U 1 1 527C458A
 P 6200 5300
-F 0 "P?" H 6200 5600 40  0000 C CNN
+F 0 "P15" H 6200 5600 40  0000 C CNN
 F 1 "CLK-" H 6200 5550 30  0000 C CNN
 F 2 "" H 6200 5300 60  0000 C CNN
@@
 $EndComp
 $Comp
-L TST P?
+L TST P16
 U 1 1 527C4599
 P 6000 5600
-F 0 "P?" H 6000 5900 40  0000 C CNN
+F 0 "P16" H 6000 5900 40  0000 C CNN
 F 1 "160Clk+" H 6000 5850 30  0000 C CNN
 F 2 "" H 6000 5600 60  0000 C CNN
@@
 $EndComp
 $Comp
-L TST P?
+L TST P17
 U 1 1 527C45A8
 P 6200 6100
-F 0 "P?" H 6200 6400 40  0000 C CNN
+F 0 "P17" H 6200 6400 40  0000 C CNN
 F 1 "160Clk-" H 6200 6350 30  0000 C CNN
 F 2 "" H 6200 6100 60  0000 C CNN
@@
 	1    0    0    -1
 $EndComp
+$Comp
+L TST P3
+U 1 1 527C4872
+P 1300 3600
+F 0 "P3" H 1300 3900 40  0000 C CNN
+F 1 "VD" H 1300 3850 30  0000 C CNN
+F 2 "" H 1300 3600 60  0000 C CNN
+F 3 "" H 1300 3600 60  0000 C CNN
+	1    1300 3600
+	0    -1   -1   0
+$EndComp
+$Comp
+L TST P2
+U 1 1 527C488B
+P 1350 3400
+F 0 "P2" H 1350 3700 40  0000 C CNN
+F 1 "3V3" H 1350 3650 30  0000 C CNN
+F 2 "" H 1350 3400 60  0000 C CNN
+F 3 "" H 1350 3400 60  0000 C CNN
+	1    1350 3400
+	1    0    0    -1
+$EndComp
+$Comp
+L TST P1
+U 1 1 527C48A6
+P 3300 1900
+F 0 "P1" H 3300 2200 40  0000 C CNN
+F 1 "VA" H 3300 2150 30  0000 C CNN
+F 2 "" H 3300 1900 60  0000 C CNN
+F 3 "" H 3300 1900 60  0000 C CNN
+	1    3300 1900
+	0    1    1    0
+$EndComp
+Connection ~ 6200 1300
+Connection ~ 6000 1600
+Connection ~ 6200 2100
+Connection ~ 6000 2400
+Connection ~ 6200 2900
+Connection ~ 6000 3200
+Connection ~ 6200 3700
+Connection ~ 3300 1900
+Connection ~ 1300 3600
+Connection ~ 1350 3400
+Connection ~ 6000 4000
+Connection ~ 6200 4500
+Connection ~ 6000 4800
+Connection ~ 6200 5300
+Connection ~ 6000 5600
+Connection ~ 6200 6100
+$Comp
+L TST P18
+U 1 1 527C48CE
+P 4800 6350
+F 0 "P18" H 4800 6650 40  0000 C CNN
+F 1 "RTD+" H 4800 6600 30  0000 C CNN
+F 2 "" H 4800 6350 60  0000 C CNN
+F 3 "" H 4800 6350 60  0000 C CNN
+	1    4800 6350
+	-1   0    0    1
+$EndComp
+$Comp
+L TST P19
+U 1 1 527C48DD
+P 4950 6700
+F 0 "P19" H 4950 7000 40  0000 C CNN
+F 1 "RTD-" H 4950 6950 30  0000 C CNN
+F 2 "" H 4950 6700 60  0000 C CNN
+F 3 "" H 4950 6700 60  0000 C CNN
+	1    4950 6700
+	1    0    0    -1
+$EndComp
+$Comp
+L TST P20
+U 1 1 527C4A35
+P 3100 4800
+F 0 "P20" H 3100 5100 40  0000 C CNN
+F 1 "GND" H 3100 5050 30  0000 C CNN
+F 2 "" H 3100 4800 60  0000 C CNN
+F 3 "" H 3100 4800 60  0000 C CNN
+	1    3100 4800
+	0    1    1    0
+$EndComp
 $EndSCHEMATC

Commit message: Schemafehler... RTD pads nicht verbunden...
Connections:
- net 3V3: now also P18.1
- net RTD-: now also P19.1
Changed lines of the file:
@@
 	0    1    1    0
 $EndComp
+Connection ~ 4800 6350
+Connection ~ 4950 6700
 $EndSCHEMATC
