File: FPix2DTB_90deg/CableAdapter.sch (KiCad schematic (older format))
At the start: 4 parts, among them J1 CONN-SMK20, J2 CONN-SMK20

Commit message: Save
Connections:
- net TBM_Out_A+ is gone; now on net TBM_OutA+: J2.1
- net TBM_Out_A- is gone; now on net TBM_OutA-: J2.3
Changed lines of the file:
@@
 $EndComp
 Text GLabel 6700 2750 0    60   Input ~ 0
-TBM_Out_A+
+TBM_OutA+
 Text Notes 7550 1900 0    60   ~ 0
 To adapter board
@@
 (new pin out)
 Text GLabel 6700 2850 0    60   Input ~ 0
-TBM_Out_A-
+TBM_OutA-
 Text GLabel 6650 3000 0    60   Output ~ 0
 VA

Commit message: Schematic finalized
Other:
- note added: "Two signals (RClk and 160MHzClk) are nor longer present on new HDI\nTf. they are not routed on the new adapter card\nSo we terminate them here (60 Ohms would match the connector saver cable's impedance)."
Changed lines of the file:
@@
 encoding utf-8
 Sheet 1 1
-Title "noname.sch"
+Title "Cable Adapter"
 Date "2 may 2014"
-Rev ""
-Comp ""
-Comment1 ""
+Rev "1"
+Comp "University of Nebraska-Lincoln"
+Comment1 "Adapter to use new module-to-DTB adapter with old HDI"
 Comment2 ""
 Comment3 ""
@@
 Connection ~ 2550 4550
 Connection ~ 2550 4650
+Text Notes 3450 5750 0    60   ~ 0
+Two signals (RClk and 160MHzClk) are nor longer present on new HDI\nTf. they are not routed on the new adapter card\nSo we terminate them here (60 Ohms would match the connector saver cable's impedance).
 $EndSCHEMATC
