File: singleroc-adapter-testbeam/singleroc-adapter-tb.sch (KiCad schematic (older format))
At the start: 24 parts, among them J1 CONN_40, J2 CONN-SCSI68, P1 CONN_2

Commit message: Rotatted adapter routed in principle. Space issues observed, need to try another approach (maybe add some space). Learned that the edge connector should be rotated the other way round - will start another PCB
Parts:
- C1, C10, C11, C2, C3, C4, C5, C6, C7, C8, C9: symbol C -> C-RESCUE-singleroc-adapter-tb
- R1, R2, R3, R4, R5, R6, R7, R8, R9: symbol R -> R-RESCUE-singleroc-adapter-tb
Changed lines of the file:
@@
 EESchema Schematic File Version 2
+LIBS:singleroc-adapter-tb-rescue
 LIBS:power
 LIBS:device
@@
 LIBS:memory
 LIBS:xilinx
-LIBS:special
 LIBS:microcontrollers
 LIBS:dsp
@@
 LIBS:valves
 LIBS:conn-scsi68
-LIBS:CableAdapter-cache
 LIBS:conn_40
 LIBS:singleroc-adapter-tb-cache
@@
 AIN2
 $Comp
-L R R4
+L R-RESCUE-singleroc-adapter-tb R4
 U 1 1 5391E4B4
 P 4700 6250
@@
 $EndComp
 $Comp
-L C C3
+L C-RESCUE-singleroc-adapter-tb C3
 U 1 1 5391E40D
 P 9400 4750
@@
 NoConn ~ 10150 4850
 $Comp
-L R R2
+L R-RESCUE-singleroc-adapter-tb R2
 U 1 1 5391E39C
 P 5000 4550
@@
 $EndComp
 $Comp
-L R R3
+L R-RESCUE-singleroc-adapter-tb R3
 U 1 1 5391E300
 P 4450 4150
@@
 AIN1
 $Comp
-L C C2
+L C-RESCUE-singleroc-adapter-tb C2
 U 1 1 5391E24E
 P 9200 3750
@@
 $EndComp
 $Comp
-L R R1
+L R-RESCUE-singleroc-adapter-tb R1
 U 1 1 5391E1C7
 P 2100 6250
@@
 AIN0
 $Comp
-L C C1
+L C-RESCUE-singleroc-adapter-tb C1
 U 1 1 5391DEE8
 P 9200 2850
@@
 $EndComp
 $Comp
-L C C6
+L C-RESCUE-singleroc-adapter-tb C6
 U 1 1 5391DE88
 P 10950 1150
@@
 $EndComp
 $Comp
-L C C4
+L C-RESCUE-singleroc-adapter-tb C4
 U 1 1 5391DE4B
 P 10600 1150
@@
 $EndComp
 $Comp
-L C C9
+L C-RESCUE-singleroc-adapter-tb C9
 U 1 1 5391DD79
 P 10950 1800
@@
 $EndComp
 $Comp
-L C C8
+L C-RESCUE-singleroc-adapter-tb C8
 U 1 1 5391DD75
 P 10600 1800
@@
 $EndComp
 $Comp
-L C C7
+L C-RESCUE-singleroc-adapter-tb C7
 U 1 1 5391DD72
 P 10250 1800
@@
 $EndComp
 $Comp
-L C C5
+L C-RESCUE-singleroc-adapter-tb C5
 U 1 1 5391DD61
 P 9850 1800
@@
 VA
 $Comp
-L C C10
+L C-RESCUE-singleroc-adapter-tb C10
 U 1 1 53D8A1B7
 P 3250 1550
@@
 $EndComp
 $Comp
-L C C11
+L C-RESCUE-singleroc-adapter-tb C11
 U 1 1 53D8A1DA
 P 2850 1550
@@
 $EndComp
 $Comp
-L R R5
+L R-RESCUE-singleroc-adapter-tb R5
 U 1 1 53D8A20F
 P 2350 1000
@@
 $EndComp
 $Comp
-L R R6
+L R-RESCUE-singleroc-adapter-tb R6
 U 1 1 53D8A244
 P 2350 1200
@@
 RTD-
 $Comp
-L R R7
+L R-RESCUE-singleroc-adapter-tb R7
 U 1 1 53D8A6E6
 P 2100 800
@@
 $EndComp
 $Comp
-L R R8
+L R-RESCUE-singleroc-adapter-tb R8
 U 1 1 53D8A6FB
 P 1650 1500
@@
 $EndComp
 $Comp
-L R R9
+L R-RESCUE-singleroc-adapter-tb R9
 U 1 1 53D8A710
 P 1850 1500
@@
 $EndComp
 $Comp
-L GND #PWR01
+L GND-RESCUE-singleroc-adapter-tb #PWR01
 U 1 1 53EA353E
 P 3300 7100
@@
 NoConn ~ 2800 5000
 $Comp
-L GND #PWR02
+L GND-RESCUE-singleroc-adapter-tb #PWR02
 U 1 1 53EA73CA
 P 9700 6750
@@
 $EndComp
 $Comp
-L GND #PWR03
+L GND-RESCUE-singleroc-adapter-tb #PWR03
 U 1 1 53EA7557
 P 8300 2950
@@
 $EndComp
 $Comp
-L GND #PWR04
+L GND-RESCUE-singleroc-adapter-tb #PWR04
 U 1 1 53EA7630
 P 9850 2050
@@
 $EndComp
 $Comp
-L GND #PWR05
+L GND-RESCUE-singleroc-adapter-tb #PWR05
 U 1 1 53EA7A4B
 P 3250 2000
@@
 $EndComp
 $Comp
-L GND #PWR06
+L GND-RESCUE-singleroc-adapter-tb #PWR06
 U 1 1 53EA7B28
 P 10600 1400
@@
 $EndComp
 $Comp
-L GND #PWR07
+L GND-RESCUE-singleroc-adapter-tb #PWR07
 U 1 1 53EA7B3C
 P 10950 1400
@@
 $EndComp
 $Comp
-L GND #PWR08
+L GND-RESCUE-singleroc-adapter-tb #PWR08
 U 1 1 53EA7D96
 P 8900 3850
@@
 $EndComp
 $Comp
-L GND #PWR09
+L GND-RESCUE-singleroc-adapter-tb #PWR09
 U 1 1 53EA7DAA
 P 9150 4900
@@
 $EndComp
 $Comp
-L GND #PWR010
+L GND-RESCUE-singleroc-adapter-tb #PWR010
 U 1 1 53EA8007
 P 10600 2050
@@
 $EndComp
 $Comp
-L GND #PWR011
+L GND-RESCUE-singleroc-adapter-tb #PWR011
 U 1 1 53EA81A1
 P 10950 2050
@@
 $EndComp
 $Comp
-L GND #PWR012
+L GND-RESCUE-singleroc-adapter-tb #PWR012
 U 1 1 53EA8333
 P 10250 2050
