File: Active-FPix/FPix2DTB_up.sch (KiCad schematic (older format))
At the start: 54 parts, among them J1 CONN-SCSI68, J2 CONN-SMK20, P10 VD, P11 CTR-, P12 CLK+, P13 CLK-, P14 GND, P15 RTD+, P16 RTD-, P3 RDa+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

Commit message: last? revision
Connections:
- net GND: now also D1.2 (K), J1.1, J1.12
- net I2C_SCL2 renamed 12C_SCL2
- net I2C_SDA2 renamed 12C_SDA2
Other:
- moved on the sheet: C1, C2, JP1, U1
