File: Active-FPix/FPix2DTB_up.kicad_pcb (KiCad board)
At the start: 4 copper layers, 100 x 40 mm, 59 parts, among them J1 CONN-SCSI68, J2 CONN-SMK20, P1 OutA+, P10 VD, P11 CTR-, P12 CLK+, P13 CLK-, P14 GND, P15 RTD+, P16 RTD-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

Commit message: last? revision
Parts:
- added R1: R, Resistors_SMD:R_0402, F.Cu at (111.4, 61.1)
- added R2: R, Resistors_SMD:R_0402, F.Cu at (111.6, 66.2)
- R3: footprint SM0402 -> Resistors_SMD:R_0402
- moved G*** 22.6 mm to (138.7, 64.8)
- moved G*** 8.54 mm to (129.4, 64.7)
- moved R3 7.96 mm to (122.2, 63.8)
- turned U3 to 270 degrees
Connections:
- net I2C_SCL2 renamed 12C_SCL2
- net I2C_SDA2 renamed 12C_SDA2
- net RTD+ renamed 3V3
- D1 pad 2: (no net) -> GND
- J1 pad 1: (no net) -> GND
- J1 pad 12: (no net) -> GND
- J1 pad 71: (no net) -> GND
- J1 pad 72: (no net) -> GND
Routing:
- net GND: track 134.2 -> 153.1 mm, vias 23 -> 26
- net SDATA1_n: track 32.5 -> 20.3 mm
- net (no net): track 10.9 -> 0.30 mm, vias 1 -> 0
- net SDATA1_p: track 24.5 -> 17.0 mm
- net 3V3: track 175.4 -> 179.2 mm
- net TBM_Out_A-: track 59.2 -> 56.2 mm
- net 2.5V: track 22.2 -> 19.4 mm, vias 5 -> 3
- net TBM_Out_A+: track 57.5 -> 56.5 mm
- net RTD-: track 35.4 -> 36.1 mm
- net VA: track 60.1 -> 59.5 mm
Other:
- board text added: "v2.0 - F. Meier, J. Kelty Aug 2015"
- board text removed: "v2.0 - F. Meier, Mai 2014"

Commit message: last? revision
Parts:
- added C6: 4.7u, SM0603, F.Cu at (110.8, 92.6)
Routing:
- net GND: track 153.1 -> 158.0 mm
- net 3V3: track 179.2 -> 175.0 mm
- net 2.5V: track 19.4 -> 21.8 mm
